Commit message: Refactor workspace and Docker setup for real hardware deployment

File: ros2_ws/src/prisma_rover_description/urdf/rover.xacro (robot description, xacro)
@@ -3,49 +3,32 @@
     <xacro:include filename="$(find prisma_rover_description)/urdf/rover_macro.xacro"/>
     <xacro:include filename="$(find prisma_rover_description)/urdf/utilities.xacro"/>
-    <xacro:include filename="$(find prisma_rover_description)/urdf/rover_gazebo.xacro"/>
     <!-- Launch Arguments -->
-    <xacro:arg name="is_sim" default="true"/>
     <xacro:arg name="namespace" default=""/>
-    <xacro:arg name="frame_prefix" default=""/>
-    <xacro:arg name="tf_prefix" default=""/>
     <xacro:arg name="camera" default="true"/>
-    <xacro:arg name="lidar_type" default="2d"/>
+    <xacro:arg name="lidar_type" default="3d"/>
     <!-- Base footprint at ground level -->
     <link name="base_footprint"/>
     <!-- Setup structural links and base joint -->
     <xacro:rover_base_frame parent_link="base_footprint"/>
-    <!-- IMU Link and Sensor -->
-    <xacro:imu_macro namespace="$(arg namespace)"/>
-    <!-- Simulation-only elements -->
-    <xacro:if value="$(arg is_sim)">
-        <xacro:rover_wheels_sim left_joint="diff_drive_l_joint" right_joint="diff_drive_r_joint"/>
-        <xacro:gazebo_diff_drive_controller left_joint="diff_drive_l_joint" right_joint="diff_drive_r_joint" namespace="$(arg namespace)"/>
-        <xacro:gazebo_wheel_contact/>
-        <!-- Load Sensors system plugin for Lidar and Camera simulation -->
-        <gazebo>
-            <plugin filename="libignition-gazebo-sensors-system.so" name="ignition::gazebo::systems::Sensors">
-                <render_engine>ogre2</render_engine>
-            </plugin>
-        </gazebo>
-        <!-- Conditionally load Lidar type -->
-        <xacro:if value="${'$(arg lidar_type)' == '2d'}">
-            <xacro:lidar_gazebo_sensor laser_frame="lidar_link" laser_topic="scan" namespace="$(arg namespace)"/>
-        </xacro:if>
-        <xacro:if value="${'$(arg lidar_type)' == '3d'}">
-            <xacro:livox_mid360_gazebo_sensor laser_frame="livox_link" laser_topic="scan_3d" namespace="$(arg namespace)"/>
-        </xacro:if>
-        <!-- Conditionally instantiate the camera in simulation -->
-        <xacro:if value="$(arg camera)">
-            <xacro:camera_gazebo camera_base_frame="camera_link" camera_topic="camera" camera_info_topic="camera_info" namespace="$(arg namespace)"/>
-        </xacro:if>
+    <!-- Wheels Description (needed for physical visualization via real /joint_states) -->
+    <xacro:rover_wheels/>
+    <!-- IMU Link and Joint (Hardware config) -->
+    <link name="imu_link"/>
+    <joint name="imu_to_payload" type="fixed">
+        <parent link="base_link"/>
+        <child link="imu_link"/>
+        <origin xyz="0 0 0" rpy="0 0 0"/>
+    </joint>
+    <!-- Physical Sensors Configuration -->
+    <!-- Conditionally load Lidar type -->
+    <xacro:if value="${'$(arg lidar_type)' == '2d'}">
+        <xacro:lidar_description laser_frame="laser_link"/>
     </xacro:if>
-    <!-- Real-hardware elements (simulation plugins are bypassed) -->
-    <xacro:unless value="$(arg is_sim)">
-        <xacro:if value="${'$(arg lidar_type)' == '2d'}">
-            <xacro:lidar_gazebo_sensor laser_frame="lidar_link" laser_topic="scan" namespace="$(arg namespace)"/>
-        </xacro:if>
-        <xacro:if value="${'$(arg lidar_type)' == '3d'}">
-            <xacro:livox_mid360_gazebo_sensor laser_frame="livox_link" laser_topic="scan_3d" namespace="$(arg namespace)"/>
-        </xacro:if>
-    </xacro:unless>
+    <xacro:if value="${'$(arg lidar_type)' == '3d'}">
+        <xacro:livox_mid360_description laser_frame="laser_link"/>
+    </xacro:if>
+    <!-- Conditionally instantiate the camera -->
+    <xacro:if value="$(arg camera)">
+        <xacro:camera_description/>
+    </xacro:if>
 </robot>

File: ros2_ws/src/prisma_rover_description/urdf/rover_macro.xacro (robot description, xacro)
@@ -24,7 +24,4 @@
     <xacro:property name="wheel_mass" value="1.25" />
     <xacro:property name="payload_z_offset" value="0.096" />
-    <!-- Include extra URDF files -->
-    <xacro:include filename="$(find prisma_rover_description)/urdf/imu.urdf" />
-    <xacro:property name="tf_prefix_val" value="$(arg tf_prefix)"/>
     <xacro:macro name="rover_base_frame" params="parent_link">
         <joint name="world_base_joint" type="fixed">
@@ -55,4 +52,22 @@
             </collision>
         </link>
+        <link name="payload_link">
+            <collision>
+                <origin xyz="0 0.0115 0.05" rpy="0 0 0" />
+                <geometry>
+                    <box size="${total_length} ${total_width - 2*track_width} 0.03"/>
+                </geometry>
+            </collision>
+            <inertial>
+                <origin xyz="-0.01 0 0" rpy="0 0 0"/>
+                <mass value="2.95" />
+                <inertia ixx="0.018398" ixy="0.0" ixz="0.0" iyy="0.04064" iyz="0.0" izz="0.05396" />
+            </inertial>
+        </link>
+        <joint name="payload_to_base" type="fixed">
+            <parent link="base_link"/>
+            <child link="payload_link"/>
+            <origin xyz="0 0 ${payload_z_offset}"/>
+        </joint>
         <link name="pole_link">
             <collision>
@@ -63,30 +78,189 @@
             </collision>
         </link>
-    </xacro:macro>
-    <link name="payload_link">
-        <collision>
-            <origin xyz="0 0.0115 0.05" rpy="0 0 0" />
-            <geometry>
-                <box size="${total_length} ${total_width - 2*track_width} 0.03"/>
-            </geometry>
-        </collision>
-        <inertial>
-            <origin xyz="-0.01 0 0" rpy="0 0 0"/>
-            <mass value="2.95" />
-            <inertia ixx="0.018398" ixy="0.0" ixz="0.0" iyy="0.04064" iyz="0.0" izz="0.05396" />
-        </inertial>
-    </link>
-    <joint name="payload_to_base" type="fixed">
-        <parent link="base_link"/>
-        <child link="payload_link"/>
-        <origin xyz="0 0 ${payload_z_offset}"/>
-    </joint>
-    <joint name="pole_to_payload" type="fixed">
-        <origin xyz="0 0 ${0.5 - total_height/2}" rpy="0 0 0"/>
-        <parent link="payload_link"/>
-        <child link="pole_link"/>
-    </joint>
-    <!-- Lidar Gazebo Sensor -->
-    <xacro:macro name="lidar_gazebo_sensor" params="laser_frame laser_topic namespace">
+        <joint name="pole_to_payload" type="fixed">
+            <origin xyz="0 0 ${0.5 - total_height/2}" rpy="0 0 0"/>
+            <parent link="payload_link"/>
+            <child link="pole_link"/>
+        </joint>
+    </xacro:macro>
+    <!-- Wheels Description (needed for physical visualization via real /joint_states) -->
+    <xacro:macro name="rover_wheels">
+        <!-- Front Right Wheel -->
+        <link name="fr_wheel_link">
+            <visual>
+                <origin xyz="0 0 0" rpy="-1.57 0 0" />
+                <geometry>
+                    <mesh filename="file://$(find prisma_rover_description)/meshes/pro_tire.obj" scale="0.5 0.5 1.0"/>
+                </geometry>
+                <material name="dark_grey">
+                    <color rgba="0.15 0.15 0.15 1.0"/>
+                </material>
+            </visual>
+            <collision>
+                <origin xyz="0 0 0" rpy="-1.57 0 0" />
+                <geometry>
+                    <cylinder radius="${total_height/2}" length="${track_width}"/>
+                </geometry>
+            </collision>
+            <inertial>
+                <origin xyz="0 0 0" rpy="0 0 0" />
+                <mass value="${wheel_mass}" />
+                <inertia ixx="0.005645" ixy="0.0" ixz="0.0" iyy="0.01008" iyz="0.0" izz="0.005645"/>
+            </inertial>
+        </link>
+        <joint name="fr_wheel_to_base" type="continuous">
+            <parent link="base_link"/>
+            <child link="fr_wheel_link"/>
+            <axis xyz="0 1 0"/>
+            <origin xyz="${wheel_x_offset + front_flipper_x_offset} ${-wheel_y_offset} 0" rpy="0 0 0"/>
+        </joint>
+        <!-- Front Left Wheel -->
+        <link name="fl_wheel_link">
+            <visual>
+                <origin xyz="0 0 0" rpy="1.57 0 0" />
+                <geometry>
+                    <mesh filename="file://$(find prisma_rover_description)/meshes/pro_tire.obj" scale="0.5 0.5 1.0"/>
+                </geometry>
+                <material name="dark_grey">
+                    <color rgba="0.15 0.15 0.15 1.0"/>
+                </material>
+            </visual>
+            <collision>
+                <origin xyz="0 0 0" rpy="1.57 0 0" />
+                <geometry>
+                    <cylinder radius="${total_height/2}" length="${track_width}"/>
+                </geometry>
+            </collision>
+            <inertial>
+                <origin xyz="0 0 0" rpy="0 0 0" />
+                <mass value="${wheel_mass}" />
+                <inertia ixx="0.005645" ixy="0.0" ixz="0.0" iyy="0.01008" iyz="0.0" izz="0.005645"/>
+            </inertial>
+        </link>
+        <joint name="fl_wheel_to_base" type="continuous">
+            <parent link="base_link"/>
+            <child link="fl_wheel_link"/>
+            <axis xyz="0 1 0"/>
+            <origin xyz="${wheel_x_offset + front_flipper_x_offset} ${wheel_y_offset} 0" rpy="0 0 0"/>
+        </joint>
+        <!-- Rear Right Wheel -->
+        <link name="rr_wheel_link">
+            <visual>
+                <origin xyz="0 0 0" rpy="1.57 0 3.1415" />
+                <geometry>
+                    <mesh filename="file://$(find prisma_rover_description)/meshes/pro_tire.obj" scale="0.5 0.5 1.0"/>
+                </geometry>
+                <material name="dark_grey">
+                    <color rgba="0.15 0.15 0.15 1.0"/>
+                </material>
+            </visual>
+            <collision>
+                <origin xyz="0 0 0" rpy="1.57 0 3.1415" />
+                <geometry>
+                    <cylinder radius="${total_height/2}" length="${track_width}"/>
+                </geometry>
+            </collision>
+            <inertial>
+                <origin xyz="0 0 0" rpy="0 0 0" />
+                <mass value="${wheel_mass}" />
+                <inertia ixx="0.005645" ixy="0.0" ixz="0.0" iyy="0.01008" iyz="0.0" izz="0.005645"/>
+            </inertial>
+        </link>
+        <joint name="rr_wheel_to_base" type="continuous">
+            <parent link="base_link"/>
+            <child link="rr_wheel_link"/>
+            <axis xyz="0 1 0"/>
+            <origin xyz="${-wheel_x_offset} ${-wheel_y_offset} 0" rpy="0 0 0"/>
+        </joint>
+        <!-- Rear Left Wheel -->
+        <link name="rl_wheel_link">
+            <visual>
+                <origin xyz="0 0 0" rpy="-1.57 0 3.1415" />
+                <geometry>
+                    <mesh filename="file://$(find prisma_rover_description)/meshes/pro_tire.obj" scale="0.5 0.5 1.0"/>
+                </geometry>
+                <material name="dark_grey">
+                    <color rgba="0.15 0.15 0.15 1.0"/>
+                </material>
+            </visual>
+            <collision>
+                <origin xyz="0 0 0" rpy="-1.57 0 3.1415" />
+                <geometry>
+                    <cylinder radius="${total_height/2}" length="${track_width}"/>
+                </geometry>
+            </collision>
+            <inertial>
+                <origin xyz="0 0 0" rpy="0 0 0" />
+                <mass value="${wheel_mass}" />
+                <inertia ixx="0.005645" ixy="0.0" ixz="0.0" iyy="0.01008" iyz="0.0" izz="0.005645"/>
+            </inertial>
+        </link>
+        <joint name="rl_wheel_to_base" type="continuous">
+            <parent link="base_link"/>
+            <child link="rl_wheel_link"/>
+            <axis xyz="0 1 0"/>
+            <origin xyz="${-wheel_x_offset} ${wheel_y_offset} 0" rpy="0 0 0"/>
+        </joint>
+    </xacro:macro>
+    <!-- IMU Description -->
+    <xacro:macro name="imu_description">
+        <link name="imu_link"/>
+        <joint name="imu_to_payload" type="fixed">
+            <parent link="base_link"/>
+            <child link="imu_link"/>
+            <origin xyz="0 0 0" rpy="0 0 0"/>
+        </joint>
+    </xacro:macro>
+    <!-- RealSense RGB-D Camera Description -->
+    <xacro:macro name="camera_description">
+        <joint name="camera_to_payload" type="fixed">
+            <origin xyz="0.22 0.0 0.15" rpy="0 0 0"/>
+            <parent link="payload_link"/>
+            <child link="camera_link"/>
+        </joint>
+        <link name="camera_link">
+            <visual>
+                <origin xyz="0 0 0" rpy="1.57 0 1.57"/>
+                <geometry>
+                    <mesh filename="file://$(find prisma_rover_description)/meshes/realsense.obj"/>
+                </geometry>
+                <material name="camera_black">
+                    <color rgba="0.2 0.2 0.2 1.0"/>
+                </material>
+            </visual>
+            <collision>
+                <origin xyz="-0.01 0.0 0.0" rpy="0 0 0"/>
+                <geometry>
+                    <box size="0.02 0.1 0.025"/>
+                </geometry>
+            </collision>
+        </link>
+        <joint name="camera_rgb_joint" type="fixed">
+            <origin xyz="0.005 0.018 0.013" rpy="0 0 0"/>
+            <parent link="camera_link"/>
+            <child link="camera_rgb_frame"/>
+        </joint>
+        <link name="camera_rgb_frame"/>
+        <joint name="camera_rgb_optical_joint" type="fixed">
+            <origin xyz="0 0 0" rpy="-1.57 0 -1.57"/>
+            <parent link="camera_rgb_frame"/>
+            <child link="camera_rgb_optical_frame"/>
+        </joint>
+        <link name="camera_rgb_optical_frame"/>
+        <joint name="camera_depth_joint" type="fixed">
+            <origin xyz="0.005 0.028 0.013" rpy="0 0 0"/>
+            <parent link="camera_link"/>
+            <child link="camera_depth_frame"/>
+        </joint>
+        <link name="camera_depth_frame"/>
+        <joint name="camera_depth_optical_joint" type="fixed">
+            <origin xyz="0 0 0" rpy="-1.57 0 -1.57"/>
+            <parent link="camera_depth_frame"/>
+            <child link="camera_depth_optical_frame"/>
+        </joint>
+        <link name="camera_depth_optical_frame"/>
+    </xacro:macro>
+    <!-- 2D RPLidar Lidar Description -->
+    <xacro:macro name="lidar_description" params="laser_frame">
         <joint name="lidar_to_payload" type="fixed">
             <parent link="payload_link"/>
@@ -111,47 +285,7 @@
             </collision>
         </link>
-        <gazebo reference="${laser_frame}">
-            <visual>
-                <material>
-                    <ambient>0.5 0.1 0.1 1.0</ambient>
-                    <diffuse>0.7 0.2 0.2 1.0</diffuse>
-                    <specular>0.6 0.6 0.6 1.0</specular>
-                </material>
-                <visibility_flags>2</visibility_flags>
-            </visual>
-            <sensor name='gpu_lidar' type='gpu_lidar'>
-                <pose>0 0 0.03 0 0 0</pose>
-                <topic>${namespace}/${laser_topic}</topic>
-                <ignition_frame_id>${tf_prefix_val}lidar_link</ignition_frame_id>
-                <update_rate>10</update_rate>
-                <lidar>
-                    <visibility_mask>4</visibility_mask>
-                    <scan>
-                        <horizontal>
-                            <samples>640</samples>
-                            <resolution>1</resolution>
-                            <min_angle>-3.14159</min_angle>
-                            <max_angle>3.14159</max_angle>
-                        </horizontal>
-                        <vertical>
-                            <samples>1</samples>
-                            <resolution>1</resolution>
-                            <min_angle>0.0</min_angle>
-                            <max_angle>0.0</max_angle>
-                        </vertical>
-                    </scan>
-                    <range>
-                        <min>0.15</min>
-                        <max>10.0</max>
-                        <resolution>0.01</resolution>
-                    </range>
-                </lidar>
-                <visualize>true</visualize>
-            </sensor>
-        </gazebo>
-    </xacro:macro>
-    <!-- Livox Mid-360 Lidar Gazebo Sensor -->
-    <!-- The physical Livox Mid-360 has a cylinder-like form factor (65mm diameter x 40mm height) -->
-    <xacro:macro name="livox_mid360_gazebo_sensor" params="laser_frame laser_topic namespace">
+    </xacro:macro>
+    <!-- 3D Livox Mid-360 Lidar Description -->
+    <xacro:macro name="livox_mid360_description" params="laser_frame">
         <joint name="livox_to_payload" type="fixed">
             <parent link="payload_link"/>
@@ -163,5 +297,5 @@
                 <origin xyz="0 0 0" rpy="0 0 0"/>
                 <geometry>
-                    <cylinder radius="0.0325" length="0.04"/> <!-- 65mm diameter, 40mm height -->
+                    <cylinder radius="0.0325" length="0.04"/>
                 </geometry>
                 <material name="dark_grey">
@@ -176,48 +310,4 @@
             </collision>
         </link>
-        <gazebo reference="${laser_frame}">
-            <visual>
-                <material>
-                    <ambient>0.5 0.1 0.1 1.0</ambient>
-                    <diffuse>0.7 0.2 0.2 1.0</diffuse>
-                    <specular>0.6 0.6 0.6 1.0</specular>
-                </material>
-                <visibility_flags>2</visibility_flags>
-            </visual>
-            <sensor name='livox_mid360' type='gpu_lidar'>
-                <pose>0 0 0.03 0 0 0</pose>
-                <topic>${namespace}/${laser_topic}</topic>
-                <ignition_frame_id>${tf_prefix_val}livox_link</ignition_frame_id>
-                <update_rate>10</update_rate> <!-- 10 Hz typical Livox scanning/spin rate -->
-                <lidar>
-                    <visibility_mask>4</visibility_mask>
-                    <scan>
-                        <horizontal>
-                            <samples>360</samples>
-                            <resolution>1</resolution>
-                            <!-- 360° Horizontal FOV -->
-                            <min_angle>-3.14159</min_angle>
-                            <max_angle>3.14159</max_angle>
-                        </horizontal>
-                        <vertical>
-                            <samples>60</samples>
-                            <resolution>1</resolution>
-                            <!-- 59° Vertical FOV: -7° (-0.122 rad) to +52° (0.907 rad) -->
-                            <min_angle>-0.122</min_angle>
-                            <max_angle>0.907</max_angle>
-                        </vertical>
-                    </scan>
-                    <range>
-                        <!-- Minimum range of 0.1m matches the physical Livox specs -->
-                        <min>0.1</min>
-                        <!-- Maximum range capped at 20m in simulation for performance/indoor bounds -->
-                        <!-- (Physical Livox Mid-360 can range up to 40m at 10% reflectivity) -->
-                        <max>20.0</max>
-                        <resolution>0.01</resolution>
-                    </range>
-                </lidar>
-                <visualize>true</visualize>
-            </sensor>
-        </gazebo>
     </xacro:macro>
 </robot>
