Commit message: Expose rviz launch flag and fix URDF mesh paths using package:// scheme

File: ros2_ws/src/prisma_rover_description/urdf/rover_macro.xacro (robot description, xacro)
@@ -34,5 +34,5 @@
                 <origin xyz="0 0 -0.035" rpy="0 0 0"/>
                 <geometry>
-                    <mesh filename="file://$(find prisma_rover_description)/meshes/prisma_rover.obj" scale="0.001 0.001 0.001"/>
+                    <mesh filename="package://prisma_rover_description/meshes/prisma_rover.obj" scale="0.001 0.001 0.001"/>
                 </geometry>
                 <material name="silver">
@@ -91,5 +91,5 @@
                 <origin xyz="0 0 0" rpy="-1.57 0 0" />
                 <geometry>
-                    <mesh filename="file://$(find prisma_rover_description)/meshes/pro_tire.obj" scale="0.5 0.5 1.0"/>
+                    <mesh filename="package://prisma_rover_description/meshes/pro_tire.obj" scale="0.5 0.5 1.0"/>
                 </geometry>
                 <material name="dark_grey">
@@ -120,5 +120,5 @@
                 <origin xyz="0 0 0" rpy="1.57 0 0" />
                 <geometry>
-                    <mesh filename="file://$(find prisma_rover_description)/meshes/pro_tire.obj" scale="0.5 0.5 1.0"/>
+                    <mesh filename="package://prisma_rover_description/meshes/pro_tire.obj" scale="0.5 0.5 1.0"/>
                 </geometry>
                 <material name="dark_grey">
@@ -149,5 +149,5 @@
                 <origin xyz="0 0 0" rpy="1.57 0 3.1415" />
                 <geometry>
-                    <mesh filename="file://$(find prisma_rover_description)/meshes/pro_tire.obj" scale="0.5 0.5 1.0"/>
+                    <mesh filename="package://prisma_rover_description/meshes/pro_tire.obj" scale="0.5 0.5 1.0"/>
                 </geometry>
                 <material name="dark_grey">
@@ -178,5 +178,5 @@
                 <origin xyz="0 0 0" rpy="-1.57 0 3.1415" />
                 <geometry>
-                    <mesh filename="file://$(find prisma_rover_description)/meshes/pro_tire.obj" scale="0.5 0.5 1.0"/>
+                    <mesh filename="package://prisma_rover_description/meshes/pro_tire.obj" scale="0.5 0.5 1.0"/>
                 </geometry>
                 <material name="dark_grey">
@@ -223,5 +223,5 @@
                 <origin xyz="0 0 0" rpy="1.57 0 1.57"/>
                 <geometry>
-                    <mesh filename="file://$(find prisma_rover_description)/meshes/realsense.obj"/>
+                    <mesh filename="package://prisma_rover_description/meshes/realsense.obj"/>
                 </geometry>
                 <material name="camera_black">
@@ -272,5 +272,5 @@
                 <origin xyz="0 0 0" rpy="-1.57 3.1415 3.1415"/>
                 <geometry>
-                    <mesh filename="file://$(find prisma_rover_description)/meshes/rplidar_s2.obj"/>
+                    <mesh filename="package://prisma_rover_description/meshes/rplidar_s2.obj"/>
                 </geometry>
                 <material name="lidar_red">

Commit message: fix: change meshes from .obj to .dae for RViz2 compatibility and add DAE mesh files

File: ros2_ws/src/prisma_rover_description/urdf/rover_macro.xacro (robot description, xacro)
@@ -34,5 +34,5 @@
                 <origin xyz="0 0 -0.035" rpy="0 0 0"/>
                 <geometry>
-                    <mesh filename="package://prisma_rover_description/meshes/prisma_rover.obj" scale="0.001 0.001 0.001"/>
+                    <mesh filename="package://prisma_rover_description/meshes/prisma_rover.dae" scale="0.001 0.001 0.001"/>
                 </geometry>
                 <material name="silver">
@@ -91,5 +91,5 @@
                 <origin xyz="0 0 0" rpy="-1.57 0 0" />
                 <geometry>
-                    <mesh filename="package://prisma_rover_description/meshes/pro_tire.obj" scale="0.5 0.5 1.0"/>
+                    <mesh filename="package://prisma_rover_description/meshes/pro_tire.dae" scale="0.5 0.5 1.0"/>
                 </geometry>
                 <material name="dark_grey">
@@ -120,5 +120,5 @@
                 <origin xyz="0 0 0" rpy="1.57 0 0" />
                 <geometry>
-                    <mesh filename="package://prisma_rover_description/meshes/pro_tire.obj" scale="0.5 0.5 1.0"/>
+                    <mesh filename="package://prisma_rover_description/meshes/pro_tire.dae" scale="0.5 0.5 1.0"/>
                 </geometry>
                 <material name="dark_grey">
@@ -149,5 +149,5 @@
                 <origin xyz="0 0 0" rpy="1.57 0 3.1415" />
                 <geometry>
-                    <mesh filename="package://prisma_rover_description/meshes/pro_tire.obj" scale="0.5 0.5 1.0"/>
+                    <mesh filename="package://prisma_rover_description/meshes/pro_tire.dae" scale="0.5 0.5 1.0"/>
                 </geometry>
                 <material name="dark_grey">
@@ -178,5 +178,5 @@
                 <origin xyz="0 0 0" rpy="-1.57 0 3.1415" />
                 <geometry>
-                    <mesh filename="package://prisma_rover_description/meshes/pro_tire.obj" scale="0.5 0.5 1.0"/>
+                    <mesh filename="package://prisma_rover_description/meshes/pro_tire.dae" scale="0.5 0.5 1.0"/>
                 </geometry>
                 <material name="dark_grey">
@@ -223,5 +223,5 @@
                 <origin xyz="0 0 0" rpy="1.57 0 1.57"/>
                 <geometry>
-                    <mesh filename="package://prisma_rover_description/meshes/realsense.obj"/>
+                    <mesh filename="package://prisma_rover_description/meshes/realsense.dae"/>
                 </geometry>
                 <material name="camera_black">
@@ -272,5 +272,5 @@
                 <origin xyz="0 0 0" rpy="-1.57 3.1415 3.1415"/>
                 <geometry>
-                    <mesh filename="package://prisma_rover_description/meshes/rplidar_s2.obj"/>
+                    <mesh filename="package://prisma_rover_description/meshes/rplidar_s2.dae"/>
                 </geometry>
                 <material name="lidar_red">

Commit message: fix: change wheel joint types to fixed and remove joint_state_publisher for physical robot bringup to resolve missing wheel TFs

File: ros2_ws/src/prisma_rover_description/urdf/rover_macro.xacro (robot description, xacro)
@@ -109,8 +109,7 @@
             </inertial>
         </link>
-        <joint name="fr_wheel_to_base" type="continuous">
+        <joint name="fr_wheel_to_base" type="fixed">
             <parent link="base_link"/>
             <child link="fr_wheel_link"/>
-            <axis xyz="0 1 0"/>
             <origin xyz="${wheel_x_offset + front_flipper_x_offset} ${-wheel_y_offset} 0" rpy="0 0 0"/>
         </joint>
@@ -138,8 +137,7 @@
             </inertial>
         </link>
-        <joint name="fl_wheel_to_base" type="continuous">
+        <joint name="fl_wheel_to_base" type="fixed">
             <parent link="base_link"/>
             <child link="fl_wheel_link"/>
-            <axis xyz="0 1 0"/>
             <origin xyz="${wheel_x_offset + front_flipper_x_offset} ${wheel_y_offset} 0" rpy="0 0 0"/>
         </joint>
@@ -167,8 +165,7 @@
             </inertial>
         </link>
-        <joint name="rr_wheel_to_base" type="continuous">
+        <joint name="rr_wheel_to_base" type="fixed">
             <parent link="base_link"/>
             <child link="rr_wheel_link"/>
-            <axis xyz="0 1 0"/>
             <origin xyz="${-wheel_x_offset} ${-wheel_y_offset} 0" rpy="0 0 0"/>
         </joint>
@@ -196,8 +193,7 @@
             </inertial>
         </link>
-        <joint name="rl_wheel_to_base" type="continuous">
+        <joint name="rl_wheel_to_base" type="fixed">
             <parent link="base_link"/>
             <child link="rl_wheel_link"/>
-            <axis xyz="0 1 0"/>
             <origin xyz="${-wheel_x_offset} ${wheel_y_offset} 0" rpy="0 0 0"/>
         </joint>
